Commit message: improve gazebo config; add mantra_with_j10

File: mantra_with_gripper_gazebo/urdf/mantra_with_gripper_description.xacro (robot description, xacro)
@@ -1,8 +1,5 @@
-<?xml version="1.0" encoding="utf-8"?>
-<!-- This URDF was automatically created by SolidWorks to URDF Exporter! Originally created by Stephen Brawner (brawner@gmail.com)
-     Commit Version: 1.5.0-0-g9aa0fdb  Build Version: 1.5.7004.21443
-     For more information, please see http://wiki.ros.org/sw_urdf_exporter -->
-<robot
-  name="mantra_with_gripper_description">
+<?xml version="1.0"?>
+<robot name="mantra_with_gripper_description" xmlns:xacro="http://ros.org/wiki/xacro">
+  <xacro:property name="M_PI" value="3.1415926536"/>
   <link
     name="base_link">
@@ -571,6 +568,8 @@
       offset="0" />
   </joint>
+  <!-- scene -->
+  <xacro:include filename="$(find mantra_with_gripper_gazebo)/urdf/scene.urdf.xacro"/>
   <!-- sensors -->
-  <include filename="$(find mantra_with_gripper_gazebo)/urdf/sensors/camera.urdf.xacro"/>
+  <xacro:include filename="$(find mantra_with_gripper_gazebo)/urdf/sensors/camera.urdf.xacro"/>
   <!-- #################################  gazebo ################################## -->
   <!-- modify EffortJointInterface to PositionJointInterface -->

File: mantra_with_j10_description/urdf/mantra_description.urdf (robot description, URDF)
Before this commit: robot mantra, 9 links, 8 joints
Links:
- removed link box
- added link bottom_link, mass 98000.55; collision box size=0 0 0; visual mesh filename=package://mantra_with_j10_description/meshes/bottom_link.STL
- added link earth_link; collision box size=0.1 0.1 0.04; visual box size=5 13 0.02
- added link plane_link; collision mesh filename=package://mantra_with_j10_description/meshes/J10B.STL; visual mesh filename=package://mantra_with_j10_description/meshes/J10B.STL
- added link top_link; collision box size=0 0 0; visual box size=5 13 0.02
- link base_link: mass 2.12515524577406 -> None; geometry collision mesh filename=package://mantra_with_j10_description/meshes/base_link.STL; visual mesh filename=package://mantra_with_j10_description/meshes/base_link.STL
- link link1: mass 0.449846417611502 -> 1111110.449846417611502; geometry collision mesh filename=package://mantra_with_j10_description/meshes/link1.STL; visual mesh filename=package://mantra_with_j10_description/meshes/link1.STL
- link link2: geometry collision mesh filename=package://mantra_with_j10_description/meshes/link2.STL; visual mesh filename=package://mantra_with_j10_description/meshes/link2.STL
- link link3: geometry collision mesh filename=package://mantra_with_j10_description/meshes/link3.STL; visual mesh filename=package://mantra_with_j10_description/meshes/link3.STL
- link link4: geometry collision mesh filename=package://mantra_with_j10_description/meshes/joint4.STL; visual mesh filename=package://mantra_with_j10_description/meshes/joint4.STL
- link link5: geometry collision mesh filename=package://mantra_with_j10_description/meshes/link5.STL; visual mesh filename=package://mantra_with_j10_description/meshes/link5.STL
- link link6: geometry collision mesh filename=package://mantra_with_j10_description/meshes/link6.STL; visual mesh filename=package://mantra_with_j10_description/meshes/link6.STL
- link link7: geometry collision mesh filename=package://mantra_with_j10_description/meshes/link7.STL; visual mesh filename=package://mantra_with_j10_description/meshes/link7.STL
Joints:
- removed joint base_to_box
- added joint base_joint: type prismatic, parent bottom_link, child base_link, origin xyz=0.065704 -0.22324 0.22 rpy=0 -4.0598E-05 1.3143, axis -4.0598E-05 0 1, limit lower=0 upper=2 effort=100 velocity=1.0
- added joint bottom_joint: type fixed, parent earth_link, child bottom_link, origin xyz=-2.19 0 0 rpy=0 0 0
- added joint bottom_joint2: type fixed, parent earth_link, child top_link, origin xyz=0 0 1.49 rpy=0 0 0
- added joint top_joint: type fixed, parent top_link, child plane_link, origin xyz=0.6 0 0.73 rpy=0 0 0
- joint joint1: limit lower=-1.5708 upper=1.5708 effort=100 velocity=1 -> lower=-3.1415 upper=3.1415 effort=100 velocity=1; origin xyz=0 0 0.2005 rpy=0 0 0 -> xyz=0.09 -0.005 0.171 rpy=0 0 0
- joint joint2: axis 0 0 -1 -> 0 0 1; limit lower=-1.85 upper=1.85 effort=100 velocity=1 -> lower=-3.1415 upper=3.1415 effort=100 velocity=1
- joint joint3: axis 0 0 -1 -> 0 0 1; limit lower=-1.5708 upper=1.5708 effort=100 velocity=1 -> lower=-3.1415 upper=3.1415 effort=100 velocity=1
- joint joint4: limit lower=-1.85 upper=1.85 effort=100 velocity=1 -> lower=-3.1415 upper=3.1415 effort=100 velocity=1
- joint joint5: limit lower=-1.5708 upper=1.5708 effort=100 velocity=1 -> lower=-3.1415 upper=3.1415 effort=100 velocity=1
- joint joint6: axis 0 0 -1 -> 0 0 1; limit lower=-1.85 upper=1.85 effort=100 velocity=1 -> lower=-3.1415 upper=3.1415 effort=100 velocity=1
- joint joint7: limit lower=-1.5708 upper=1.5708 effort=100 velocity=1 -> lower=-3.1415 upper=3.1415 effort=100 velocity=1
