Commit message: add some package for mantra_with_oil_gun

File: mantra_with_gripper_gazebo/urdf/mantra_with_gripper_description.xacro (robot description, xacro)
@@ -8,5 +8,5 @@
         xyz="5.69641035035705E-08 -7.52429850161379E-09 0.0534781808387783"
         rpy="0 0 0" />
-      <mass value="500" />  <!-- modified -->
+      <mass value="5" />  <!-- modified -->
       <!-- modified -->
       <inertia
@@ -51,10 +51,10 @@
         value="0.449846417611502" />
       <inertia
-        ixx="0.00281542194513947"
-        ixy="-2.97928363529203E-08"
-        ixz="2.31552459198658E-09"
-        iyy="0.00237879024815951"
-        iyz="-0.000689611051918419"
-        izz="0.00161666621542504" />
+        ixx="1.0"
+        ixy="0.0"
+        ixz="0.0"
+        iyy="1.0"
+        iyz="0.0"
+        izz="1.0" />
     </inertial>
     <visual>
@@ -109,10 +109,10 @@
         value="0.449846417611509" />
       <inertia
-        ixx="0.00281542194513949"
-        ixy="-2.3155245922964E-09"
-        ixz="-2.97928363554505E-08"
-        iyy="0.00161666621542506"
-        iyz="0.000689611051918419"
-        izz="0.00237879024815952" />
+        ixx="1.0"
+        ixy="0.0"
+        ixz="0.0"
+        iyy="1.0"
+        iyz="0.0"
+        izz="1.0" />
     </inertial>
     <visual>
@@ -167,10 +167,10 @@
         value="0.392582340089193" />
       <inertia
-        ixx="0.0020755242879527"
-        ixy="1.39339603463947E-08"
-        ixz="-2.854811113402E-08"
-        iyy="0.00178702026485436"
-        iyz="-0.000503155834932376"
-        izz="0.00121405044233485" />
+        ixx="1.0"
+        ixy="0.0"
+        ixz="0.0"
+        iyy="1.0"
+        iyz="0.0"
+        izz="1.0" />
     </inertial>
     <visual>
@@ -225,10 +225,10 @@
         value="0.367226253241491" />
       <inertia
-        ixx="0.00189945127986856"
-        ixy="1.10761786473211E-08"
-        ixz="-3.7570793904099E-09"
-        iyy="0.00102605162314097"
-        iyz="0.000467411288512599"
-        izz="0.00163165412446067" />
+        ixx="1.0"
+        ixy="0.0"
+        ixz="0.0"
+        iyy="1.0"
+        iyz="0.0"
+        izz="1.0" />
     </inertial>
     <visual>
@@ -283,10 +283,10 @@
         value="0.367226254016741" />
       <inertia
-        ixx="0.00189945125870264"
-        ixy="-3.75974500932253E-09"
-        ixz="-1.10613008672603E-08"
-        iyy="0.00163165410820963"
-        iyz="-0.000467411240126133"
-        izz="0.00102605163568241" />
+        ixx="1.0"
+        ixy="0.0"
+        ixz="0.0"
+        iyy="1.0"
+        iyz="0.0"
+        izz="1.0" />
     </inertial>
     <visual>
@@ -340,11 +340,11 @@
       <mass
         value="0.367226253239117" />
-      <inertia
-        ixx="0.00189945137374859"
-        ixy="1.10879827352058E-08"
-        ixz="-3.81500844090566E-09"
-        iyy="0.00102605167941246"
-        iyz="0.000467411315869438"
-        izz="0.00163165420801843" />
+      <<inertia
+        ixx="1.0"
+        ixy="0.0"
+        ixz="0.0"
+        iyy="1.0"
+        iyz="0.0"
+        izz="1.0" />
     </inertial>
     <visual>
@@ -399,10 +399,10 @@
         value="0.14043817532843" />
       <inertia
-        ixx="0.000166560052257127"
-        ixy="2.71160607993557E-20"
-        ixz="-8.59213210250315E-20"
-        iyy="0.000166602712740968"
-        iyz="2.78725555163462E-08"
-        izz="0.000232492320290339" />
+        ixx="1.0"
+        ixy="0.0"
+        ixz="0.0"
+        iyy="1.0"
+        iyz="0.0"
+        izz="1.0" />
     </inertial>
     <visual>
@@ -457,10 +457,10 @@
         value="0.00194999999999999" />
       <inertia
-        ixx="1.50312499999997E-07"
-        ixy="6.61485086202342E-25"
-        ixz="1.48998375260736E-23"
-        iyy="1.73712499999997E-07"
-        iyz="-4.21006794862361E-25"
-        izz="3.15249999999998E-08" />
+        ixx="1.0"
+        ixy="0.0"
+        ixz="0.0"
+        iyy="1.0"
+        iyz="0.0"
+        izz="1.0" />
     </inertial>
     <visual>
@@ -515,10 +515,10 @@
         value="0.00194999999999999" />
       <inertia
-        ixx="1.50312499999997E-07"
-        ixy="6.61485086202342E-25"
-        ixz="1.48998375260736E-23"
-        iyy="1.73712499999997E-07"
-        iyz="-4.21006794862361E-25"
-        izz="3.15249999999998E-08" />
+        ixx="1.0"
+        ixy="0.0"
+        ixz="0.0"
+        iyy="1.0"
+        iyz="0.0"
+        izz="1.0" />
     </inertial>
     <visual>

File: mantra_with_gripper_gazebo/urdf/scene.urdf.xacro (robot description, xacro)
@@ -3,9 +3,8 @@
     <!-- ///////////////  oil_filler1  /////////////// -->
     <joint name="oil_filler_joint" type="fixed">
-        <origin xyz="1.15 0.2 1.0" rpy="0 ${-M_PI/2} 0"/>
+        <origin xyz="1.0 0.0 1.0" rpy="0 ${-M_PI/2} 0"/>
         <parent link="base_link"/>
         <child link="oil_filler_link"/>
     </joint>
-    <!-- oil_filler -->
     <link name="oil_filler_link">
         <collision>
@@ -34,10 +33,9 @@
     </gazebo>
     <!-- ///////////////  oil_filler2  /////////////// -->
-    <joint name="oil_filler_joint2" type="fixed">
-        <origin xyz="1.15 -0.2 1.2" rpy="0 ${-M_PI/2} 0"/>
+    <!-- <joint name="oil_filler_joint2" type="fixed">
+        <origin xyz="0.9 -0.2 1.2" rpy="0 ${-M_PI/2} 0"/>
         <parent link="base_link"/>
         <child link="oil_filler_link2"/>
     </joint>
-    <!-- oil_filler2 -->
     <link name="oil_filler_link2">
         <collision>
@@ -52,5 +50,4 @@
             <mesh filename="package://mantra_with_gripper_gazebo/meshes/oil_filler.STL" />
             </geometry>
-            <!-- <material name="red"/> -->
         </visual>
         <inertial>
@@ -64,5 +61,5 @@
     <gazebo reference="oil_filler_link2">
         <material>Gazebo/WhiteGlow</material>
-    </gazebo>
+    </gazebo> -->
     <!-- ///////////////  background  /////////////// -->
     <joint name="background_joint" type="fixed">

File: mantra_with_oil_gun_description/urdf/mantra_with_oil_gun_description.urdf (robot description, URDF)
Before this commit: robot mantra, 9 links, 8 joints
Links:
- removed link box
- added link oil_gun_link, mass 4.65959936378476; collision mesh filename=package://mantra_with_gripper_gazebo/meshes/oil_gun.STL; visual mesh filename=package://mantra_with_gripper_gazebo/meshes/oil_gun.STL
- link base_link: mass 2.12515524577406 -> None; geometry collision mesh filename=package://mantra_with_oil_gun_description/meshes/base_link.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; visual mesh filename=package://mantra_with_oil_gun_description/meshes/base_link.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
- link link1: geometry collision mesh filename=package://mantra_with_oil_gun_description/meshes/link1.STL; visual mesh filename=package://mantra_with_oil_gun_description/meshes/link1.STL
- link link2: geometry collision mesh filename=package://mantra_with_oil_gun_description/meshes/link2.STL; visual mesh filename=package://mantra_with_oil_gun_description/meshes/link2.STL
- link link3: geometry collision mesh filename=package://mantra_with_oil_gun_description/meshes/link3.STL; visual mesh filename=package://mantra_with_oil_gun_description/meshes/link3.STL
- link link4: geometry collision mesh filename=package://mantra_with_oil_gun_description/meshes/link4.STL; visual mesh filename=package://mantra_with_oil_gun_description/meshes/link4.STL
- link link5: mass 0.36722625401674 -> 0.367226254016741; geometry collision mesh filename=package://mantra_with_oil_gun_description/meshes/link5.STL; visual mesh filename=package://mantra_with_oil_gun_description/meshes/link5.STL
- link link6: geometry collision mesh filename=package://mantra_with_oil_gun_description/meshes/link6.STL; visual mesh filename=package://mantra_with_oil_gun_description/meshes/link6.STL
- link link7: geometry collision mesh filename=package://mantra_with_oil_gun_description/meshes/link7.STL; visual mesh filename=package://mantra_with_oil_gun_description/meshes/link7.STL
Joints:
- removed joint base_to_box
- added joint oil_gun_joint: type fixed, parent link7, child oil_gun_link, origin xyz=0 0 0.0655 rpy=1.5708 0 0, axis 0 0 0, limit lower=-1.85 upper=1.85 effort=100 velocity=1

File: mantra_with_oil_gun_gazebo/urdf/mantra_with_oil_gun_description.xacro (robot description, xacro)
@@ -1,8 +1,5 @@
-<?xml version="1.0" encoding="utf-8"?>
-<!-- This URDF was automatically created by SolidWorks to URDF Exporter! Originally created by Stephen Brawner (brawner@gmail.com)
-     Commit Version: 1.5.0-0-g9aa0fdb  Build Version: 1.5.7004.21443
-     For more information, please see http://wiki.ros.org/sw_urdf_exporter -->
-<robot
-  name="mantra_with_gripper_description">
+<?xml version="1.0"?>
+<robot name="mantra_with_oil_gun_description" xmlns:xacro="http://ros.org/wiki/xacro">
+  <xacro:property name="M_PI" value="3.1415926536" />
   <link
     name="base_link">
@@ -11,5 +8,5 @@
         xyz="5.69641035035705E-08 -7.52429850161379E-09 0.0534781808387783"
         rpy="0 0 0" />
-      <mass value="500" />  <!-- modified -->
+      <mass value="5" />  <!-- modified -->
       <!-- modified -->
       <inertia
@@ -27,19 +24,19 @@
       <geometry>
         <mesh
-          filename="package://mantra_with_gripper_description/meshes/base_link.STL" />
-      </geometry>
-      <material
-        name="">
-        <color
-          rgba="1 1 1 1" />
-      </material>
-    </visual>
-    <collision>
-      <origin
-        xyz="0 0 0"
-        rpy="0 0 0" />
-      <geometry>
-        <mesh
-          filename="package://mantra_with_gripper_description/meshes/base_link.STL" />
+          filename="package://mantra_with_oil_gun_description/meshes/base_link.STL" />
+      </geometry>
+      <material
+        name="">
+        <color
+          rgba="1 1 1 1" />
+      </material>
+    </visual>
+    <collision>
+      <origin
+        xyz="0 0 0"
+        rpy="0 0 0" />
+      <geometry>
+        <mesh
+          filename="package://mantra_with_oil_gun_description/meshes/base_link.STL" />
       </geometry>
     </collision>
@@ -54,32 +51,32 @@
         value="0.449846417611502" />
       <inertia
-        ixx="0.00281542194513947"
-        ixy="-2.97928363529203E-08"
-        ixz="2.31552459198658E-09"
-        iyy="0.00237879024815951"
-        iyz="-0.000689611051918419"
-        izz="0.00161666621542504" />
-    </inertial>
-    <visual>
-      <origin
-        xyz="0 0 0"
-        rpy="0 0 0" />
-      <geometry>
-        <mesh
-          filename="package://mantra_with_gripper_description/meshes/link1.STL" />
-      </geometry>
-      <material
-        name="">
-        <color
-          rgba="1 1 1 1" />
-      </material>
-    </visual>
-    <collision>
-      <origin
-        xyz="0 0 0"
-        rpy="0 0 0" />
-      <geometry>
-        <mesh
-          filename="package://mantra_with_gripper_description/meshes/link1.STL" />
+        ixx="1.0"
+        ixy="0.0"
+        ixz="0.0"
+        iyy="1.0"
+        iyz="0.0"
+        izz="1.0" />
+    </inertial>
+    <visual>
+      <origin
+        xyz="0 0 0"
+        rpy="0 0 0" />
+      <geometry>
+        <mesh
+          filename="package://mantra_with_oil_gun_description/meshes/link1.STL" />
+      </geometry>
+      <material
+        name="">
+        <color
+          rgba="1 1 1 1" />
+      </material>
+    </visual>
+    <collision>
+      <origin
+        xyz="0 0 0"
+        rpy="0 0 0" />
+      <geometry>
+        <mesh
+          filename="package://mantra_with_oil_gun_description/meshes/link1.STL" />
       </geometry>
     </collision>
@@ -112,32 +109,32 @@
         value="0.449846417611509" />
       <inertia
-        ixx="0.00281542194513949"
-        ixy="-2.3155245922964E-09"
-        ixz="-2.97928363554505E-08"
-        iyy="0.00161666621542506"
-        iyz="0.000689611051918419"
-        izz="0.00237879024815952" />
-    </inertial>
-    <visual>
-      <origin
-        xyz="0 0 0"
-        rpy="0 0 0" />
-      <geometry>
-        <mesh
-          filename="package://mantra_with_gripper_description/meshes/link2.STL" />
-      </geometry>
-      <material
-        name="">
-        <color
-          rgba="1 1 1 1" />
-      </material>
-    </visual>
-    <collision>
-      <origin
-        xyz="0 0 0"
-        rpy="0 0 0" />
-      <geometry>
-        <mesh
-          filename="package://mantra_with_gripper_description/meshes/link2.STL" />
+        ixx="1.0"
+        ixy="0.0"
+        ixz="0.0"
+        iyy="1.0"
+        iyz="0.0"
+        izz="1.0" />
+    </inertial>
+    <visual>
+      <origin
+        xyz="0 0 0"
+        rpy="0 0 0" />
+      <geometry>
+        <mesh
+          filename="package://mantra_with_oil_gun_description/meshes/link2.STL" />
+      </geometry>
+      <material
+        name="">
+        <color
+          rgba="1 1 1 1" />
+      </material>
+    </visual>
+    <collision>
+      <origin
+        xyz="0 0 0"
+        rpy="0 0 0" />
+      <geometry>
+        <mesh
+          filename="package://mantra_with_oil_gun_description/meshes/link2.STL" />
       </geometry>
     </collision>
@@ -170,32 +167,32 @@
         value="0.392582340089193" />
       <inertia
-        ixx="0.0020755242879527"
-        ixy="1.39339603463947E-08"
-        ixz="-2.854811113402E-08"
-        iyy="0.00178702026485436"
-        iyz="-0.000503155834932376"
-        izz="0.00121405044233485" />
-    </inertial>
-    <visual>
-      <origin
-        xyz="0 0 0"
-        rpy="0 0 0" />
-      <geometry>
-        <mesh
-          filename="package://mantra_with_gripper_description/meshes/link3.STL" />
-      </geometry>
-      <material
-        name="">
-        <color
-          rgba="1 1 1 1" />
-      </material>
-    </visual>
-    <collision>
-      <origin
-        xyz="0 0 0"
-        rpy="0 0 0" />
-      <geometry>
-        <mesh
-          filename="package://mantra_with_gripper_description/meshes/link3.STL" />
+        ixx="1.0"
+        ixy="0.0"
+        ixz="0.0"
+        iyy="1.0"
+        iyz="0.0"
+        izz="1.0" />
+    </inertial>
+    <visual>
+      <origin
+        xyz="0 0 0"
+        rpy="0 0 0" />
+      <geometry>
+        <mesh
+          filename="package://mantra_with_oil_gun_description/meshes/link3.STL" />
+      </geometry>
+      <material
+        name="">
+        <color
+          rgba="1 1 1 1" />
+      </material>
+    </visual>
+    <collision>
+      <origin
+        xyz="0 0 0"
+        rpy="0 0 0" />
+      <geometry>
+        <mesh
+          filename="package://mantra_with_oil_gun_description/meshes/link3.STL" />
       </geometry>
     </collision>
@@ -228,32 +225,32 @@
         value="0.367226253241491" />
       <inertia
-        ixx="0.00189945127986856"
-        ixy="1.10761786473211E-08"
-        ixz="-3.7570793904099E-09"
-        iyy="0.00102605162314097"
-        iyz="0.000467411288512599"
-        izz="0.00163165412446067" />
-    </inertial>
-    <visual>
-      <origin
-        xyz="0 0 0"
-        rpy="0 0 0" />
-      <geometry>
-        <mesh
-          filename="package://mantra_with_gripper_description/meshes/link4.STL" />
-      </geometry>
-      <material
-        name="">
-        <color
-          rgba="1 1 1 1" />
-      </material>
-    </visual>
-    <collision>
-      <origin
-        xyz="0 0 0"
-        rpy="0 0 0" />
-      <geometry>
-        <mesh
-          filename="package://mantra_with_gripper_description/meshes/link4.STL" />
+        ixx="1.0"
+        ixy="0.0"
+        ixz="0.0"
+        iyy="1.0"
+        iyz="0.0"
+        izz="1.0" />
+    </inertial>
+    <visual>
+      <origin
+        xyz="0 0 0"
+        rpy="0 0 0" />
+      <geometry>
+        <mesh
+          filename="package://mantra_with_oil_gun_description/meshes/link4.STL" />
+      </geometry>
+      <material
+        name="">
+        <color
+          rgba="1 1 1 1" />
+      </material>
+    </visual>
+    <collision>
+      <origin
+        xyz="0 0 0"
+        rpy="0 0 0" />
+      <geometry>
+        <mesh
+          filename="package://mantra_with_oil_gun_description/meshes/link4.STL" />
       </geometry>
     </collision>
@@ -286,32 +283,32 @@
         value="0.367226254016741" />
       <inertia
-        ixx="0.00189945125870264"
-        ixy="-3.75974500932253E-09"
-        ixz="-1.10613008672603E-08"
-        iyy="0.00163165410820963"
-        iyz="-0.000467411240126133"
-        izz="0.00102605163568241" />
-    </inertial>
-    <visual>
-      <origin
-        xyz="0 0 0"
-        rpy="0 0 0" />
-      <geometry>
-        <mesh
-          filename="package://mantra_with_gripper_description/meshes/link5.STL" />
-      </geometry>
-      <material
-        name="">
-        <color
-          rgba="1 1 1 1" />
-      </material>
-    </visual>
-    <collision>
-      <origin
-        xyz="0 0 0"
-        rpy="0 0 0" />
-      <geometry>
-        <mesh
-          filename="package://mantra_with_gripper_description/meshes/link5.STL" />
+        ixx="1.0"
+        ixy="0.0"
+        ixz="0.0"
+        iyy="1.0"
+        iyz="0.0"
+        izz="1.0" />
+    </inertial>
+    <visual>
+      <origin
+        xyz="0 0 0"
+        rpy="0 0 0" />
+      <geometry>
+        <mesh
+          filename="package://mantra_with_oil_gun_description/meshes/link5.STL" />
+      </geometry>
+      <material
+        name="">
+        <color
+          rgba="1 1 1 1" />
+      </material>
+    </visual>
+    <collision>
+      <origin
+        xyz="0 0 0"
+        rpy="0 0 0" />
+      <geometry>
+        <mesh
+          filename="package://mantra_with_oil_gun_description/meshes/link5.STL" />
       </geometry>
     </collision>
@@ -344,32 +341,32 @@
         value="0.367226253239117" />
       <inertia
-        ixx="0.00189945137374859"
-        ixy="1.10879827352058E-08"
-        ixz="-3.81500844090566E-09"
-        iyy="0.00102605167941246"
-        iyz="0.000467411315869438"
-        izz="0.00163165420801843" />
-    </inertial>
-    <visual>
-      <origin
-        xyz="0 0 0"
-        rpy="0 0 0" />
-      <geometry>
-        <mesh
-          filename="package://mantra_with_gripper_description/meshes/link6.STL" />
-      </geometry>
-      <material
-        name="">
-        <color
-          rgba="1 1 1 1" />
-      </material>
-    </visual>
-    <collision>
-      <origin
-        xyz="0 0 0"
-        rpy="0 0 0" />
-      <geometry>
-        <mesh
-          filename="package://mantra_with_gripper_description/meshes/link6.STL" />
+        ixx="1.0"
+        ixy="0.0"
+        ixz="0.0"
+        iyy="1.0"
+        iyz="0.0"
+        izz="1.0" />
+    </inertial>
+    <visual>
+      <origin
+        xyz="0 0 0"
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