Commit message: add mantra with yinshi gripper description; change 1.5708 to 1.5707963267949 in urdf

File: mantra_description/urdf/mantra_with_box_description.urdf (robot description, URDF)
Before this commit: robot mantra_with_oil_gun_description, 9 links, 8 joints
Links:
- removed link oil_gun_link
- added link box; visual box size=0.1 0.1 0.1
- link base_link: mass None -> 2.12515524577406; geometry collision mesh filename=package://mantra_description/meshes/base_link.STL; visual mesh filename=package://mantra_description/meshes/base_link.STL
- link link1: geometry collision mesh filename=package://mantra_description/meshes/link1.STL; visual mesh filename=package://mantra_description/meshes/link1.STL
- link link2: geometry collision mesh filename=package://mantra_description/meshes/link2.STL; visual mesh filename=package://mantra_description/meshes/link2.STL
- link link3: geometry collision mesh filename=package://mantra_description/meshes/link3.STL; visual mesh filename=package://mantra_description/meshes/link3.STL
- link link4: geometry collision mesh filename=package://mantra_description/meshes/link4.STL; visual mesh filename=package://mantra_description/meshes/link4.STL
- link link5: mass 0.367226254016741 -> 0.36722625401674; geometry collision mesh filename=package://mantra_description/meshes/link5.STL; visual mesh filename=package://mantra_description/meshes/link5.STL
- link link6: geometry collision mesh filename=package://mantra_description/meshes/link6.STL; visual mesh filename=package://mantra_description/meshes/link6.STL
- link link7: geometry collision mesh filename=package://mantra_description/meshes/link7.STL; visual mesh filename=package://mantra_description/meshes/link7.STL
Joints:
- removed joint oil_gun_joint
- added joint base_to_box: type fixed, parent base_link, child box, origin xyz=0.88 0.0 0.546 rpy=0 0 0

File: mantra_description/urdf/mantra_with_robotiq_gripper_description.urdf (robot description, URDF)
Before this commit: robot mantra_with_oil_gun_description, 9 links, 8 joints
Links:
- removed link oil_gun_link
- added link gripper, mass 4.65959936378476; collision mesh filename=package://mantra_description/meshes/robotiq_gripper.STL; visual mesh filename=package://mantra_description/meshes/robotiq_gripper.STL
- link base_link: mass None -> 2.12515524577406; geometry collision mesh filename=package://mantra_description/meshes/base_link.STL; visual mesh filename=package://mantra_description/meshes/base_link.STL
- link link1: geometry collision mesh filename=package://mantra_description/meshes/link1.STL; visual mesh filename=package://mantra_description/meshes/link1.STL
- link link2: geometry collision mesh filename=package://mantra_description/meshes/link2.STL; visual mesh filename=package://mantra_description/meshes/link2.STL
- link link3: geometry collision mesh filename=package://mantra_description/meshes/link3.STL; visual mesh filename=package://mantra_description/meshes/link3.STL
- link link4: geometry collision mesh filename=package://mantra_description/meshes/link4.STL; visual mesh filename=package://mantra_description/meshes/link4.STL
- link link5: mass 0.367226254016741 -> 0.36722625401674; geometry collision mesh filename=package://mantra_description/meshes/link5.STL; visual mesh filename=package://mantra_description/meshes/link5.STL
- link link6: geometry collision mesh filename=package://mantra_description/meshes/link6.STL; visual mesh filename=package://mantra_description/meshes/link6.STL
- link link7: geometry collision mesh filename=package://mantra_description/meshes/link7.STL; visual mesh filename=package://mantra_description/meshes/link7.STL
Joints:
- removed joint oil_gun_joint
- added joint gripper: type fixed, parent link7, child gripper, origin xyz=0 0 0.0655 rpy=0 0 0, axis 0 0 0, limit lower=-1.85 upper=1.85 effort=100 velocity=1

File: mantra_with_gripper_description/urdf/mantra_with_gripper_description.urdf (robot description, URDF)
Before this commit: robot mantra_with_gripper_description, 10 links, 9 joints
Joints:
- joint joint2: origin xyz=0 0 0.17 rpy=1.5708 0 0 -> xyz=0 0 0.17 rpy=1.5707963267949 0 0
- joint joint3: origin xyz=0 0.17 0 rpy=-1.5708 0 0 -> xyz=0 0.17 0 rpy=-1.5707963267949 0 0
- joint joint4: origin xyz=0 0 0.16 rpy=1.5708 0 0 -> xyz=0 0 0.16 rpy=1.5707963267949 0 0
- joint joint5: origin xyz=0 0.16 0 rpy=-1.5708 0 0 -> xyz=0 0.16 0 rpy=-1.5707963267949 0 0
- joint joint6: origin xyz=0 0 0.16 rpy=1.5708 0 0 -> xyz=0 0 0.16 rpy=1.5707963267949 0 0
- joint joint7: origin xyz=0 0.2255 0 rpy=-1.5708 0 0 -> xyz=0 0.2255 0 rpy=-1.5707963267949 0 0

File: mantra_with_gripper_gazebo/urdf/mantra_with_gripper_description.xacro (robot description, xacro)
@@ -340,5 +340,5 @@
       <mass
         value="0.367226253239117" />
-      <<inertia
+      <inertia
         ixx="1.0"
         ixy="0.0"

File: mantra_with_gripper_gazebo/urdf/sensors/camera.urdf.xacro (robot description, xacro)
@@ -8,8 +8,8 @@
         <origin xyz="-0.1 0.0 0.0" rpy="0 ${-M_PI/2} 0"/>
         <parent link="link7"/>
-        <child link="camera_link"/>
+        <child link="camera_color_optical_frame"/>
    </joint>
    <!-- Camera -->
-   <link name="camera_link">
+   <link name="camera_color_optical_frame">
        <collision>
            <origin xyz="0 0 0" rpy="${-M_PI} 0 ${M_PI/2}"/>

File: mantra_with_gripper_gazebo/urdf/sensors/depth_camera.gazebo.xacro (robot description, xacro)
@@ -4,5 +4,5 @@
 <robot name="camera" xmlns:xacro="http://ros.org/wiki/xacro">
 <!-- camera -->
-  <gazebo reference="camera_link">
+  <gazebo reference="camera_color_optical_frame">
     <!-- <material>Gazebo/Red</material> -->
     <sensor type="depth" name="camera">
@@ -25,9 +25,9 @@
         <cameraName>camera</cameraName>
         <imageTopicName>color/image_raw</imageTopicName>
-        <depthImageTopicName>depth/image_raw</depthImageTopicName>
-        <pointCloudTopicName>depth/points</pointCloudTopicName>
-        <cameraInfoTopicName>camera_info</cameraInfoTopicName>
-        <depthImageCameraInfoTopicName>depth/camera_info</depthImageCameraInfoTopicName>
-        <frameName>camera_link</frameName>
+        <depthImageTopicName>aligned_depth_to_color/image_raw</depthImageTopicName>
+        <pointCloudTopicName>aligned_depth_to_color/points</pointCloudTopicName>
+        <cameraInfoTopicName>color/camera_info</cameraInfoTopicName>
+        <depthImageCameraInfoTopicName>aligned_depth_to_color/camera_info</depthImageCameraInfoTopicName>
+        <frameName>camera_color_optical_frame</frameName>
         <Baseline>0.2</Baseline>
         <distortionK1>0</distortionK1>

File: mantra_with_j10_description/urdf/mantra_description.urdf (robot description, URDF)
Before this commit: robot mantra_with_j10_description, 12 links, 11 joints
Joints:
- joint joint2: origin xyz=0 0 0.17 rpy=1.5708 0 0 -> xyz=0 0 0.17 rpy=1.5707963267949 0 0
- joint joint3: origin xyz=0 0.17 0 rpy=-1.5708 0 0 -> xyz=0 0.17 0 rpy=-1.5707963267949 0 0
- joint joint4: origin xyz=0 0 0.16 rpy=1.5708 0 0 -> xyz=0 0 0.16 rpy=1.5707963267949 0 0
- joint joint5: origin xyz=0 0.16 0 rpy=-1.5708 0 0 -> xyz=0 0.16 0 rpy=-1.5707963267949 0 0
- joint joint6: origin xyz=0 0 0.16 rpy=1.5708 0 0 -> xyz=0 0 0.16 rpy=1.5707963267949 0 0
- joint joint7: origin xyz=0 0.16 0 rpy=-1.5708 0 0 -> xyz=0 0.16 0 rpy=-1.5707963267949 0 0
