Commit message: add controllers.yaml

File: mantra_description/urdf/mantra_description.urdf (robot description, URDF)
Before this commit: robot mantra_description, 9 links, 8 joints
Joints:
- joint joint1: limit lower=-3.1415 upper=3.1415 effort=100 velocity=1 -> lower=-1.5708 upper=1.5708 effort=100 velocity=1

Commit message: fix the bug of joint4/link4 and modify the joint limits

File: mantra_description/urdf/mantra_description.urdf (robot description, URDF)
Before this commit: robot mantra_description, 9 links, 8 joints
Links:
- removed link joint4
- added link link4, mass 0.367226253241491; collision mesh filename=package://mantra_description/meshes/joint4.STL; visual mesh filename=package://mantra_description/meshes/joint4.STL
Joints:
- joint gripper: limit lower=-1.5708 upper=1.5708 effort=100 velocity=1 -> lower=-1.9 upper=1.9 effort=100 velocity=1
- joint joint2: limit lower=-1.5708 upper=1.5708 effort=100 velocity=1 -> lower=-1.9 upper=1.9 effort=100 velocity=1
- joint joint4: child joint4 -> link4; limit lower=-1.5708 upper=1.5708 effort=100 velocity=1 -> lower=-1.9 upper=1.9 effort=100 velocity=1
- joint joint5: parent joint4 -> link4
- joint joint6: limit lower=-1.5708 upper=1.5708 effort=100 velocity=1 -> lower=-1.9 upper=1.9 effort=100 velocity=1

Commit message: robot could move by moveit! now

File: mantra_description/urdf/mantra_description.urdf (robot description, URDF)
Before this commit: robot mantra_description, 9 links, 8 joints
Joints:
- joint joint2: axis 0 0 1 -> 0 0 -1
- joint joint3: axis 0 0 1 -> 0 0 -1
- joint joint6: axis 0 0 1 -> 0 0 -1

Commit message: Add pyqt5 project; Add another node for joint motion

File: mantra_description/urdf/mantra_description.urdf (robot description, URDF)
Before this commit: robot mantra_description, 9 links, 8 joints
Joints:
- joint gripper: limit lower=-1.9 upper=1.9 effort=100 velocity=1 -> lower=-1.85 upper=1.85 effort=100 velocity=1
- joint joint2: limit lower=-1.9 upper=1.9 effort=100 velocity=1 -> lower=-1.85 upper=1.85 effort=100 velocity=1
- joint joint4: limit lower=-1.9 upper=1.9 effort=100 velocity=1 -> lower=-1.85 upper=1.85 effort=100 velocity=1
- joint joint6: limit lower=-1.9 upper=1.9 effort=100 velocity=1 -> lower=-1.85 upper=1.85 effort=100 velocity=1

Commit message: use mantra to pick up juggle

File: mantra_description/urdf/mantra_description.urdf (robot description, URDF)
Before this commit: robot mantra_description, 9 links, 8 joints
Joints:
- joint joint7: limit lower=-3.1415 upper=3.1415 effort=100 velocity=1 -> lower=-1.5708 upper=1.5708 effort=100 velocity=1

Commit message: add gripper, ee_joint type: prismatic, use mimic in urdf to make two ee_joint move at the same time

File: mantra_description/urdf/mantra_description.urdf (robot description, URDF)
Before this commit: robot mantra_description, 9 links, 8 joints
Links:
- removed link gripper
- added link ee_link1, mass 0.00194999999999999; collision mesh filename=package://mantra_description/meshes/ee_link1.STL; visual mesh filename=package://mantra_description/meshes/ee_link1.STL
- added link ee_link2, mass 0.00194999999999999; collision mesh filename=package://mantra_description/meshes/ee_link2.STL; visual mesh filename=package://mantra_description/meshes/ee_link2.STL
- link link4: geometry collision mesh filename=package://mantra_description/meshes/link4.STL; visual mesh filename=package://mantra_description/meshes/link4.STL
- link link5: mass 0.36722625401674 -> 0.367226254016741
Joints:
- removed joint gripper
- added joint ee_joint1: type prismatic, parent link7, child ee_link1, origin xyz=0 0 0.126 rpy=0 0 0, axis 0 -1 0, limit lower=0 upper=0.04 effort=0 velocity=0
- added joint ee_joint2: type prismatic, parent link7, child ee_link2, origin xyz=0 0 0.126 rpy=0 0 0, axis 0 1 0, limit lower=-0.04 upper=0 effort=0 velocity=0, mimic joint=ee_joint1 multiplier=1 offset=0
- joint joint7: origin xyz=0 0.16 0 rpy=-1.5708 0 0 -> xyz=0 0.2255 0 rpy=-1.5708 0 0

Commit message: add mantra_with_gripper description and moveit config

File: mantra_description/urdf/mantra_description.urdf (robot description, URDF)
Before this commit: robot mantra_description, 10 links, 9 joints
Links:
- removed link ee_link1
- removed link ee_link2
- added link gripper, mass 4.65959936378476; collision mesh filename=package://mantra_description/meshes/gripper.STL; visual mesh filename=package://mantra_description/meshes/gripper.STL
- link link4: geometry collision mesh filename=package://mantra_description/meshes/joint4.STL; visual mesh filename=package://mantra_description/meshes/joint4.STL
- link link5: mass 0.367226254016741 -> 0.36722625401674
Joints:
- removed joint ee_joint1
- removed joint ee_joint2
- added joint gripper: type fixed, parent link7, child gripper, origin xyz=0 0 0.0655 rpy=0 0 0, axis 0 0 0, limit lower=-1.85 upper=1.85 effort=100 velocity=1
- joint joint7: origin xyz=0 0.2255 0 rpy=-1.5708 0 0 -> xyz=0 0.16 0 rpy=-1.5708 0 0

Commit message: add package:mantra_with_gripper_gazebo

File: mantra_description/urdf/mantra_description.urdf (robot description, URDF)
Before this commit: robot mantra_description, 9 links, 8 joints
Links:
- link base_link: mass None -> 2.12515524577406

File: mantra_with_gripper_gazebo/urdf/mantra_with_gripper_description.urdf (robot description, URDF)
Before this commit: robot mantra_with_gripper_description, 10 links, 9 joints
Links:
- link base_link: mass None -> 500

Commit message: use mantra move service in hmi

File: mantra_description/urdf/mantra_description.urdf (robot description, URDF)
Before this commit: robot mantra, 8 links, 7 joints
Joints:
- joint joint2: limit lower=-1.5708 upper=1.5708 effort=0 velocity=0 -> lower=-1.900 upper=1.900 effort=0 velocity=0
- joint joint4: limit lower=-1.5708 upper=1.5708 effort=0 velocity=0 -> lower=-1.900 upper=1.900 effort=0 velocity=0
- joint joint6: limit lower=-1.5708 upper=1.5708 effort=0 velocity=0 -> lower=-1.900 upper=1.900 effort=0 velocity=0

File: mantra_with_j10_description/urdf/mantra_description.urdf (robot description, URDF)
Before this commit: robot mantra_with_j10_description, 12 links, 11 joints
Joints:
- joint top_joint: origin xyz=0.6 0 0.73 rpy=0 0 0 -> xyz=0.5 0.5 0.73 rpy=0 0 0

Commit message: add pose controller to mantra hmi

File: mantra_description/urdf/mantra_description.urdf (robot description, URDF)
Before this commit: robot mantra, 8 links, 7 joints
Joints:
- joint joint2: limit lower=-1.900 upper=1.900 effort=0 velocity=0 -> lower=-1.930 upper=1.930 effort=0 velocity=0
- joint joint4: limit lower=-1.900 upper=1.900 effort=0 velocity=0 -> lower=-1.880 upper=1.880 effort=0 velocity=0
- joint joint6: limit lower=-1.900 upper=1.900 effort=0 velocity=0 -> lower=-1.930 upper=1.930 effort=0 velocity=0

Commit message: show pose in hmi realtime; change lower/upper from 1.57 to 3.0 in urdf

File: mantra_description/urdf/mantra_description.urdf (robot description, URDF)
Before this commit: robot mantra, 8 links, 7 joints
Joints:
- joint joint1: limit lower=-1.5708 upper=1.5708 effort=0 velocity=0 -> lower=-3.0 upper=3.0 effort=0 velocity=0
- joint joint3: limit lower=-1.5708 upper=1.5708 effort=0 velocity=0 -> lower=-3.0 upper=3.0 effort=0 velocity=0
- joint joint5: limit lower=-1.5708 upper=1.5708 effort=0 velocity=0 -> lower=-3.0 upper=3.0 effort=0 velocity=0
- joint joint7: limit lower=-1.5708 upper=1.5708 effort=0 velocity=0 -> lower=-3.0 upper=3.0 effort=0 velocity=0

Commit message: update mantra description and test hand ey calibration

File: mantra_description/urdf/mantra_description.urdf (robot description, URDF)
Before this commit: robot mantra, 8 links, 7 joints
Links:
- added link ee_link
- link base_link: geometry collision mesh filename=package://mantra_description/meshes/base_link.STL; visual mesh filename=package://mantra_description/meshes/visual/base_link.STL
- link link1: mass 0.449846417611502 -> 0.44985; geometry collision mesh filename=package://mantra_description/meshes/link1.STL; visual mesh filename=package://mantra_description/meshes/visual/link1.STL
- link link2: mass 0.449846417611509 -> 0.44985; geometry collision mesh filename=package://mantra_description/meshes/link2.STL; visual mesh filename=package://mantra_description/meshes/visual/link2.STL
- link link3: mass 0.392582340089193 -> 0.39258; geometry collision mesh filename=package://mantra_description/meshes/link3.STL; visual mesh filename=package://mantra_description/meshes/visual/link3.STL
- link link4: mass 0.367226253241491 -> 0.36723; geometry collision mesh filename=package://mantra_description/meshes/link4.STL; visual mesh filename=package://mantra_description/meshes/visual/link4.STL
- link link5: mass 0.36722625401674 -> 0.36723; geometry collision mesh filename=package://mantra_description/meshes/link5.STL; visual mesh filename=package://mantra_description/meshes/visual/link5.STL
- link link6: mass 0.367226253239117 -> 0.36723; geometry collision mesh filename=package://mantra_description/meshes/link6.STL; visual mesh filename=package://mantra_description/meshes/visual/link6.STL
- link link7: mass 0.271729140017722 -> 0.14044; geometry collision mesh filename=package://mantra_description/meshes/link7.STL; visual mesh filename=package://mantra_description/meshes/visual/link7.STL
Joints:
- added joint ee_joint: type fixed, parent link7, child ee_link, origin xyz=0 0 0.0655 rpy=0 0 0, axis 0 0 0
- joint joint3: axis 0 0 1 -> 0 0 -1
- joint joint5: origin xyz=0 0.223720996230328 0 rpy=-1.5707963267949 0 0 -> xyz=0 0.16 0 rpy=-1.5707963267949 0 0
- joint joint6: origin xyz=0 0 0.096279003769672 rpy=1.5707963267949 0 0 -> xyz=0 0 0.16 rpy=1.5707963267949 0 0
- joint joint7: origin xyz=0 0.2255 0 rpy=-1.5707963267949 0 0 -> xyz=0 0.16 0 rpy=-1.5707963267949 0 0
