Commit message: tsdf fusion looks well now

File: mantra_description/urdf/mantra.urdf (robot description, URDF)
Before this commit: robot mantra, 9 links, 8 joints
Links:
- link ee_link: mass None -> 0.13129; geometry collision mesh filename=package://mantra_description/meshes/collision/ee_link.STL; visual mesh filename=package://mantra_description/meshes/visual/ee_link.STL

Commit message: test pick up object use gpd; add cal_obj_pose_in_world function

File: mantra_description/urdf/mantra.urdf (robot description, URDF)
Before this commit: robot mantra, 9 links, 8 joints
Joints:
- joint joint7: limit lower=-3.0 upper=3.0 effort=0 velocity=0 -> lower=-3.5 upper=3.5 effort=0 velocity=0

Commit message: get stamped images of some poses when run tsdf fusion

File: mantra_description/urdf/mantra.urdf (robot description, URDF)
Before this commit: robot mantra, 9 links, 8 joints
Links:
- added link camera, mass 0.00001; collision mesh filename=package://mantra_with_gripper_gazebo/meshes/d435.STL; visual mesh filename=package://mantra_with_gripper_gazebo/meshes/d435.STL
Joints:
- added joint camera_joint: type fixed, parent link7, child camera, origin xyz=0.0 -0.08 0.05 rpy=1.57 0 3.14
