Commit message: use multiprocessing for pointcloud create

File: mantra_with_oil_gun_gazebo/urdf/sensors/camera.urdf.xacro (robot description, xacro)
@@ -6,5 +6,5 @@
         <!-- <origin xyz="0.3 0 0.7" rpy="0 ${M_PI/2} 0"/> -->
         <!-- <parent link="base_link"/> -->
-        <origin xyz="-0.1 0.0 0.0" rpy="0 ${-M_PI/2} 0"/>
+        <origin xyz="0.1 0.0 0.0" rpy="0 ${-M_PI/2} 0"/>
         <parent link="link7"/>
         <child link="camera_link"/>
