Commit message: handeye calibration auto move and sample (use easy_handeye server to compute result)

File: mantra_gazebo/urdf/mantra_description.xacro (robot description, xacro)
@@ -500,9 +500,9 @@
     <axis
       xyz="0 0 0" />
-    <limit
+    <!-- <limit
       lower="-1.85"
       upper="1.85"
       effort="100"
-      velocity="1" />
+      velocity="1" /> -->
   </joint>
   <!-- scene -->

File: mantra_gazebo/urdf/sensors/camera.gazebo.xacro (robot description, xacro)
@@ -10,5 +10,5 @@
       <update_rate>30.0</update_rate>
       <camera name="d435i">
-        <horizontal_fov>1.047198</horizontal_fov>
+        <horizontal_fov>1.0</horizontal_fov>
         <!-- <horizontal_fov>0.95</horizontal_fov> -->
         <image>
@@ -27,5 +27,5 @@
                channels, which at that point lie in the range [0,1]. -->
           <mean>0.0</mean>
-          <stddev>0.007</stddev>
+          <stddev>0.000</stddev> <!-- 0.007 -->
         </noise>
       </camera>
@@ -37,5 +37,5 @@
         <cameraInfoTopicName>color/camera_info</cameraInfoTopicName>
         <frameName>camera_link_optical</frameName>
-        <hackBaseline>0.07</hackBaseline>
+        <hackBaseline>0.0</hackBaseline>  <!-- 0.07 -->
         <distortionK1>0.0</distortionK1>
         <distortionK2>0.0</distortionK2>

File: mantra_gazebo/urdf/sensors/camera.urdf.xacro (robot description, xacro)
@@ -26,11 +26,16 @@
            </geometry>
            <!-- <material name="red"/> -->
+           <material
+            name="">
+            <color
+            rgba="1 1 1 1" />
+           </material>
        </visual>
        <inertial>
         <mass value="0.00001" />
         <origin xyz="0 0 0" />
-        <inertia ixx="1.0" ixy="0.0" ixz="0.0"
-          iyy="1.0" iyz="0.0"
-          izz="1.0" />
+        <inertia
+            ixx="1.0" ixy="0.0" ixz="0.0"
+            iyy="1.0" iyz="0.0" izz="1.0" />
        </inertial>
    </link>

Commit message: fix some bug of mantra_gazebo; analysis calib data

File: mantra_gazebo/urdf/mantra_description.xacro (robot description, xacro)
@@ -2,4 +2,10 @@
 <robot name="mantra" xmlns:xacro="http://ros.org/wiki/xacro">
   <xacro:property name="M_PI" value="3.1415926536"/>
+  <!-- Used for fixing robot to Gazebo 'base_link' -->
+  <link name="world"/>
+  <joint name="fixed" type="fixed">
+    <parent link="world"/>
+    <child link="base_link"/>
+  </joint>
   <link
     name="base_link">
@@ -8,5 +14,5 @@
         xyz="5.69641035035705E-08 -7.52429850161379E-09 0.0534781808387783"
         rpy="0 0 0" />
-      <mass value="5" />  <!-- modified -->
+      <mass value="50" />  <!-- modified -->
       <!-- modified -->
       <inertia
@@ -97,5 +103,5 @@
       lower="-3.0"
       upper="3.0"
-      effort="0"
+      effort="100"
       velocity="1" />
   </joint>
@@ -155,5 +161,5 @@
       lower="-1.930"
       upper="1.930"
-      effort="0"
+      effort="100"
       velocity="1" />
   </joint>
@@ -213,5 +219,5 @@
       lower="-3.0"
       upper="3.0"
-      effort="0"
+      effort="100"
       velocity="1" />
   </joint>
@@ -271,5 +277,5 @@
       lower="-1.880"
       upper="1.880"
-      effort="0"
+      effort="100"
       velocity="1" />
   </joint>
@@ -329,5 +335,5 @@
       lower="-3.0"
       upper="3.0"
-      effort="0"
+      effort="100"
       velocity="1" />
   </joint>
@@ -387,5 +393,5 @@
       lower="-1.930"
       upper="1.930"
-      effort="0"
+      effort="100"
       velocity="1" />
   </joint>
@@ -445,5 +451,5 @@
       lower="-3.5"
       upper="3.5"
-      effort="0"
+      effort="100"
       velocity="1" />
   </joint>
@@ -455,5 +461,5 @@
         rpy="0 0 0" />
       <mass
-        value="0.13129" />
+        value="0.013129" />
       <inertia
         ixx="1.0"
@@ -500,9 +506,9 @@
     <axis
       xyz="0 0 0" />
-    <!-- <limit
+    <limit
       lower="-1.85"
       upper="1.85"
       effort="100"
-      velocity="1" /> -->
+      velocity="1" />
   </joint>
   <!-- scene -->
